Commit message: Upping commit

File: urdf/obj_recognition.urdf.xacro (robot description, xacro)
@@ -44,8 +44,8 @@
       <origin xyz="0 0 0" rpy="0 0 0"/>
       <geometry>
-        <box size="${width2} ${width2} ${length2}"/>
+        <box size="${width1} ${width1} ${length1}"/>
       </geometry>
-      <material name="white">
-        <color rgba="1.0 1.0 1.0 1.0"/>
+      <material name="blue">
+        <color rgba="0.0 0.0 0.8 1.0"/>
       </material>
     </visual>
@@ -53,16 +53,41 @@
       <origin xyz="0 0 0" rpy="0 0 0"/>
       <geometry>
-        <box size="${width2} ${width2} ${length2}"/>
+        <box size="${width1} ${width1} ${length1}"/>
       </geometry>
     </collision>
     <inertial>
       <origin xyz="0 0 0" rpy="0 0 0"/>
-      <mass value="${mass2}"/>
+      <mass value="${mass1}"/>
       <inertia
-        ixx="${mass2 / 12.0 * (width2*width2 + length2*length2)}" ixy="0.0" ixz="0.0"
-        iyy="${mass2 / 12.0 * (length2*length2 + width2*width2)}" iyz="0.0"
-        izz="${mass2 / 12.0 * (width2*width2 + width2*width2)}"/>
+              ixx="${mass1 / 12.0 * (width1*width1 + length1*length1)}" ixy="0.0" ixz="0.0"
+              iyy="${mass1 / 12.0 * (length1*length1 + width1*width1)}" iyz="0.0"
+              izz="${mass1 / 12.0 * (width1*width1 + width1*width1)}"/>
     </inertial>
   </link>
+  <!--<link name="link_2">-->
+    <!--<visual>-->
+      <!--<origin xyz="0 0 0" rpy="0 0 0"/>-->
+      <!--<geometry>-->
+        <!--<box size="${width2} ${width2} ${length2}"/>-->
+      <!--</geometry>-->
+      <!--<material name="white">-->
+        <!--<color rgba="1.0 1.0 1.0 1.0"/>-->
+      <!--</material>-->
+    <!--</visual>-->
+    <!--<collision>-->
+      <!--<origin xyz="0 0 0" rpy="0 0 0"/>-->
+      <!--<geometry>-->
+        <!--<box size="${width2} ${width2} ${length2}"/>-->
+      <!--</geometry>-->
+    <!--</collision>-->
+    <!--<inertial>-->
+      <!--<origin xyz="0 0 0" rpy="0 0 0"/>-->
+      <!--<mass value="${mass2}"/>-->
+      <!--<inertia-->
+        <!--ixx="${mass2 / 12.0 * (width2*width2 + length2*length2)}" ixy="0.0" ixz="0.0"-->
+        <!--iyy="${mass2 / 12.0 * (length2*length2 + width2*width2)}" iyz="0.0"-->
+        <!--izz="${mass2 / 12.0 * (width2*width2 + width2*width2)}"/>-->
+    <!--</inertial>-->
+  <!--</link>-->
   <!-- RGBD camera -->
   <link name="camera_link">

Commit message: Added correctly working urdf for robot

File: urdf/obj_recognition.urdf.xacro (robot description, xacro)
@@ -44,8 +44,8 @@
       <origin xyz="0 0 0" rpy="0 0 0"/>
       <geometry>
-        <box size="${width1} ${width1} ${length1}"/>
+        <box size="${width2} ${width2} ${length2}"/>
       </geometry>
-      <material name="blue">
-        <color rgba="0.0 0.0 0.8 1.0"/>
+      <material name="white">
+        <color rgba="1.0 1.0 1.0 1.0"/>
       </material>
     </visual>
@@ -53,41 +53,16 @@
       <origin xyz="0 0 0" rpy="0 0 0"/>
       <geometry>
-        <box size="${width1} ${width1} ${length1}"/>
+        <box size="${width2} ${width2} ${length2}"/>
       </geometry>
     </collision>
     <inertial>
       <origin xyz="0 0 0" rpy="0 0 0"/>
-      <mass value="${mass1}"/>
+      <mass value="${mass2}"/>
       <inertia
-              ixx="${mass1 / 12.0 * (width1*width1 + length1*length1)}" ixy="0.0" ixz="0.0"
-              iyy="${mass1 / 12.0 * (length1*length1 + width1*width1)}" iyz="0.0"
-              izz="${mass1 / 12.0 * (width1*width1 + width1*width1)}"/>
+        ixx="${mass2 / 12.0 * (width2*width2 + length2*length2)}" ixy="0.0" ixz="0.0"
+        iyy="${mass2 / 12.0 * (length2*length2 + width2*width2)}" iyz="0.0"
+        izz="${mass2 / 12.0 * (width2*width2 + width2*width2)}"/>
     </inertial>
   </link>
-  <!--<link name="link_2">-->
-    <!--<visual>-->
-      <!--<origin xyz="0 0 0" rpy="0 0 0"/>-->
-      <!--<geometry>-->
-        <!--<box size="${width2} ${width2} ${length2}"/>-->
-      <!--</geometry>-->
-      <!--<material name="white">-->
-        <!--<color rgba="1.0 1.0 1.0 1.0"/>-->
-      <!--</material>-->
-    <!--</visual>-->
-    <!--<collision>-->
-      <!--<origin xyz="0 0 0" rpy="0 0 0"/>-->
-      <!--<geometry>-->
-        <!--<box size="${width2} ${width2} ${length2}"/>-->
-      <!--</geometry>-->
-    <!--</collision>-->
-    <!--<inertial>-->
-      <!--<origin xyz="0 0 0" rpy="0 0 0"/>-->
-      <!--<mass value="${mass2}"/>-->
-      <!--<inertia-->
-        <!--ixx="${mass2 / 12.0 * (width2*width2 + length2*length2)}" ixy="0.0" ixz="0.0"-->
-        <!--iyy="${mass2 / 12.0 * (length2*length2 + width2*width2)}" iyz="0.0"-->
-        <!--izz="${mass2 / 12.0 * (width2*width2 + width2*width2)}"/>-->
-    <!--</inertial>-->
-  <!--</link>-->
   <!-- RGBD camera -->
   <link name="camera_link">
@@ -116,15 +91,13 @@
     <origin xyz="0 0 ${length1/2}" rpy="0 0 0"/>
   </joint>
-  <joint name="pan_joint" type="continuous">
+  <joint name="pan_joint" type="fixed">
     <parent link="link_1"/>
     <child link="link_2"/>
-    <axis xyz="0 0 1"/>
     <origin xyz="0 0 ${length1/2+length2/2}" rpy="0 0 -${pi/2}"/>
   </joint>
-  <joint name="tilt_joint" type="continuous">
+  <joint name="tilt_joint" type="fixed">
     <origin xyz="0.05 0 ${length2/2+0.02}" rpy="0 0.5 0" />
     <parent link="link_2" />
     <child link="camera_link" />
-    <axis xyz="0 1 0"/>
   </joint>
   <link name="camera_rgb_frame" />
